Commit message: Add urchin for loading URDFs

File: real_robot/assets/descriptions/xarm7_d435.urdf (robot description, URDF)
Before this commit: robot xarm7, 27 links, 25 joints
Joints:
- added joint drive_joint: type revolute, parent xarm_gripper_base_link, child left_outer_knuckle, origin xyz=0 0.035 0.059098 rpy=0 0 0, axis 1 0 0, limit lower=0 upper=0.85 effort=50 velocity=2
