Commit message: Fix xarm7_pris_finger urdf limit

File: real_robot/assets/descriptions/xarm7_pris_finger.urdf (robot description, URDF)
Before this commit: robot xarm7, 14 links, 13 joints
Joints:
- joint left_finger_joint: axis 0 0.9631963 -0.26879897 -> 0 0.96221329 -0.27229686; limit lower=0 upper=0.0446430 effort=50 velocity=0.5 -> lower=0 upper=0.0453556139430441 effort=50 velocity=0.5; origin xyz=0 0.027 0.113 rpy=0 0 0 -> xyz=0 0.02682323 0.11348719 rpy=0 0 0
- joint right_finger_joint: axis 0. -0.9631963 -0.26879897 -> 0. -0.96221329 -0.27229686; limit lower=0 upper=0.0446430 effort=50 velocity=0.5 -> lower=0 upper=0.0453556139430441 effort=50 velocity=0.5; origin xyz=0 -0.027 0.113 rpy=0 0 0 -> xyz=0 -0.02682323 0.11348719 rpy=0 0 0

File: real_robot/assets/descriptions/xarm7_pris_finger_d435.urdf (robot description, URDF)
Before this commit: robot xarm7, 23 links, 22 joints
Joints:
- joint left_finger_joint: axis 0 0.9631963 -0.26879897 -> 0 0.96221329 -0.27229686; limit lower=0 upper=0.0446430 effort=50 velocity=0.5 -> lower=0 upper=0.0453556139430441 effort=50 velocity=0.5; origin xyz=0 0.027 0.113 rpy=0 0 0 -> xyz=0 0.02682323 0.11348719 rpy=0 0 0
- joint right_finger_joint: axis 0. -0.9631963 -0.26879897 -> 0. -0.96221329 -0.27229686; limit lower=0 upper=0.0446430 effort=50 velocity=0.5 -> lower=0 upper=0.0453556139430441 effort=50 velocity=0.5; origin xyz=0 -0.027 0.113 rpy=0 0 0 -> xyz=0 -0.02682323 0.11348719 rpy=0 0 0
