Commit message: Add xarm7 urdf with reversed gripper joints; Rename to _orig.urdf

File: real_robot/assets/descriptions/xarm7.urdf (robot description, URDF)
Before this commit: robot xarm7, 18 links, 17 joints
Joints:
- joint drive_joint: axis 1 0 0 -> -1 0 0; origin xyz=0 0.035 0.059098 rpy=0 0 0 -> xyz=0 0.035 0.059098 rpy=0.85 0 0
- joint left_finger_joint: axis -1 0 0 -> 1 0 0; origin xyz=0 0.035465 0.042039 rpy=0 0 0 -> xyz=0 0.035465 0.042039 rpy=-0.85 0 0
- joint left_inner_knuckle_joint: axis 1 0 0 -> -1 0 0; origin xyz=0 0.02 0.074098 rpy=0 0 0 -> xyz=0 0.02 0.074098 rpy=0.85 0 0
- joint right_finger_joint: axis 1 0 0 -> -1 0 0; origin xyz=0 -0.035465 0.042039 rpy=0 0 0 -> xyz=0 -0.035465 0.042039 rpy=0.85 0 0
- joint right_inner_knuckle_joint: axis -1 0 0 -> 1 0 0; origin xyz=0 -0.02 0.074098 rpy=0 0 0 -> xyz=0 -0.02 0.074098 rpy=-0.85 0 0
- joint right_outer_knuckle_joint: axis -1 0 0 -> 1 0 0; origin xyz=0 -0.035 0.059098 rpy=0 0 0 -> xyz=0 -0.035 0.059098 rpy=-0.85 0 0

File: real_robot/assets/descriptions/xarm7_d435_orig.urdf (robot description, URDF)
Before this commit: robot xarm7, 27 links, 26 joints
Joints:
- joint drive_joint: axis -1 0 0 -> 1 0 0; origin xyz=0 0.035 0.059098 rpy=0.85 0 0 -> xyz=0 0.035 0.059098 rpy=0 0 0
- joint left_finger_joint: axis 1 0 0 -> -1 0 0; origin xyz=0 0.035465 0.042039 rpy=-0.85 0 0 -> xyz=0 0.035465 0.042039 rpy=0 0 0
- joint left_inner_knuckle_joint: axis -1 0 0 -> 1 0 0; origin xyz=0 0.02 0.074098 rpy=0.85 0 0 -> xyz=0 0.02 0.074098 rpy=0 0 0
- joint right_finger_joint: axis -1 0 0 -> 1 0 0; origin xyz=0 -0.035465 0.042039 rpy=0.85 0 0 -> xyz=0 -0.035465 0.042039 rpy=0 0 0
- joint right_inner_knuckle_joint: axis 1 0 0 -> -1 0 0; origin xyz=0 -0.02 0.074098 rpy=-0.85 0 0 -> xyz=0 -0.02 0.074098 rpy=0 0 0
- joint right_outer_knuckle_joint: axis 1 0 0 -> -1 0 0; origin xyz=0 -0.035 0.059098 rpy=-0.85 0 0 -> xyz=0 -0.035 0.059098 rpy=0 0 0

File: real_robot/assets/descriptions/xarm7_orig.urdf (robot description, URDF)
Before this commit: robot xarm7, 27 links, 26 joints
Links:
- removed link camera_color_frame
- removed link camera_color_optical_frame
- removed link camera_depth_frame
- removed link camera_depth_optical_frame
- removed link camera_left_ir_frame
- removed link camera_left_ir_optical_frame
- removed link camera_link
- removed link camera_right_ir_frame
- removed link camera_right_ir_optical_frame
- link link_eef: geometry 
Joints:
- removed joint camera_color_joint
- removed joint camera_color_optical_joint
- removed joint camera_depth_joint
- removed joint camera_depth_optical_joint
- removed joint camera_left_ir_joint
- removed joint camera_left_ir_optical_joint
- removed joint camera_link_joint
- removed joint camera_right_ir_joint
- removed joint camera_right_ir_optical_joint
- joint drive_joint: axis -1 0 0 -> 1 0 0; origin xyz=0 0.035 0.059098 rpy=0.85 0 0 -> xyz=0 0.035 0.059098 rpy=0 0 0
- joint gripper_fix: origin xyz=0 0 0.005 rpy=0 0 0 -> xyz=0 0 0 rpy=0 0 0
- joint left_finger_joint: axis 1 0 0 -> -1 0 0; origin xyz=0 0.035465 0.042039 rpy=-0.85 0 0 -> xyz=0 0.035465 0.042039 rpy=0 0 0
- joint left_inner_knuckle_joint: axis -1 0 0 -> 1 0 0; origin xyz=0 0.02 0.074098 rpy=0.85 0 0 -> xyz=0 0.02 0.074098 rpy=0 0 0
- joint right_finger_joint: axis -1 0 0 -> 1 0 0; origin xyz=0 -0.035465 0.042039 rpy=0.85 0 0 -> xyz=0 -0.035465 0.042039 rpy=0 0 0
- joint right_inner_knuckle_joint: axis 1 0 0 -> -1 0 0; origin xyz=0 -0.02 0.074098 rpy=-0.85 0 0 -> xyz=0 -0.02 0.074098 rpy=0 0 0
- joint right_outer_knuckle_joint: axis 1 0 0 -> -1 0 0; origin xyz=0 -0.035 0.059098 rpy=-0.85 0 0 -> xyz=0 -0.035 0.059098 rpy=0 0 0
